File: Mainboard.kicad_sch (KiCad schematic)
At the start: 4 parts

Commit message: Complete layout
Parts:
- H1, H2, H3, H4: footprint MountingHole:MountingHole_3.2mm_M3_DIN965_Pad -> mainboard:MountingHole
Changed lines of the file:
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@@
 			)
 		)
-		(property "Footprint" "MountingHole:MountingHole_3.2mm_M3_DIN965_Pad"
+		(property "Footprint" "mainboard:MountingHole"
 			(at 26.67 179.07 0)
 			(effects
@@
 			)
 		)
-		(property "Footprint" "MountingHole:MountingHole_3.2mm_M3_DIN965_Pad"
+		(property "Footprint" "mainboard:MountingHole"
 			(at 26.67 184.15 0)
 			(effects
@@
 			)
 		)
-		(property "Footprint" "MountingHole:MountingHole_3.2mm_M3_DIN965_Pad"
+		(property "Footprint" "mainboard:MountingHole"
 			(at 26.67 173.99 0)
 			(effects
@@
 			)
 		)
-		(property "Footprint" "MountingHole:MountingHole_3.2mm_M3_DIN965_Pad"
+		(property "Footprint" "mainboard:MountingHole"
 			(at 26.67 168.91 0)
 			(effects

Commit message: Updated Mounting Holes
Parts:
- H1, H2, H3, H4: footprint mainboard:MountingHole -> mainboard:MountingHole2
Changed lines of the file:
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@@
 			)
 		)
-		(property "Footprint" "mainboard:MountingHole"
+		(property "Footprint" "mainboard:MountingHole2"
 			(at 26.67 179.07 0)
 			(effects
@@
 			)
 		)
-		(property "Footprint" "mainboard:MountingHole"
+		(property "Footprint" "mainboard:MountingHole2"
 			(at 26.67 184.15 0)
 			(effects
@@
 			)
 		)
-		(property "Footprint" "mainboard:MountingHole"
+		(property "Footprint" "mainboard:MountingHole2"
 			(at 26.67 173.99 0)
 			(effects
@@
 			)
 		)
-		(property "Footprint" "mainboard:MountingHole"
+		(property "Footprint" "mainboard:MountingHole2"
 			(at 26.67 168.91 0)
 			(effects

Commit message: v1.1 Schematic
Parts:
- H1, H2, H3, H4: now left out of the parts list
Changed lines of the file:
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@@
 		(unit 1)
 		(exclude_from_sim no)
-		(in_bom yes)
+		(in_bom no)
 		(on_board yes)
 		(dnp no)
@@
 		(property "DNI" "DNI"
 			(at 26.67 179.07 0)
+			(effects
+				(font
+					(size 1.27 1.27)
+				)
+				(hide yes)
+			)
+		)
+		(property "exclude_from_bom" ""
+			(at 205.74 205.74 0)
 			(effects
 				(font
@@
 		(unit 1)
 		(exclude_from_sim no)
-		(in_bom yes)
+		(in_bom no)
 		(on_board yes)
 		(dnp no)
@@
 		(property "DNI" "DNI"
 			(at 26.67 184.15 0)
+			(effects
+				(font
+					(size 1.27 1.27)
+				)
+				(hide yes)
+			)
+		)
+		(property "exclude_from_bom" ""
+			(at 210.82 210.82 0)
 			(effects
 				(font
@@
 		(unit 1)
 		(exclude_from_sim no)
-		(in_bom yes)
+		(in_bom no)
 		(on_board yes)
 		(dnp no)
@@
 		(property "DNI" "DNI"
 			(at 26.67 173.99 0)
+			(effects
+				(font
+					(size 1.27 1.27)
+				)
+				(hide yes)
+			)
+		)
+		(property "exclude_from_bom" ""
+			(at 200.66 200.66 0)
 			(effects
 				(font
@@
 		(unit 1)
 		(exclude_from_sim no)
-		(in_bom yes)
+		(in_bom no)
 		(on_board yes)
 		(dnp no)
@@
 			(effects
 				(font
+					(size 1.27 1.27)
+				)
+				(hide yes)
+			)
+		)
+		(property "exclude_from_bom" ""
+			(at 195.58 195.58 0)
+			(effects
+				(font
