File: Peripherals.kicad_sch (KiCad schematic)
At the start: 27 parts, among them J1 Conn_02x05_Odd_Even, J13 USB_C_Receptacle_USB2.0, J16 1985807, J17 1985807, J18 1985807, J24 Micro_SD_Card_Det2, J28 USB_C_Receptacle_USB2.0, J3 1985807, J4 1985807, U10 USBLC6-2SC6, U7 USBLC6-2SC6

Commit message: Complete layout
Parts:
- removed C62: 4.7nF, Capacitor_SMD:C_0603_1608Metric, symbol Device:C_Small
- removed J3, J4: 1985807, mainboard:SCREWTERMINAL-3.5MM-2_LOCK, symbol mainboard:M023.5MM_LOCK
- removed R100, R147, R148, R91: 22R, Resistor_SMD:R_0603_1608Metric, symbol Device:R_Small
- removed R102: 1M, Resistor_SMD:R_0603_1608Metric, symbol Device:R_Small
- added C31: 47uF, Capacitor_SMD:C_0805_2012Metric, symbol Device:C_Small
- added C32: 0.1uF, Capacitor_SMD:C_0603_1608Metric, symbol Device:C_Small
- added J2: 282834-4, mainboard:TE_282834-4, symbol Connector_Generic:Conn_01x04
- J1: renamed from J13; footprint mainboard:USB_C_Receptacle_XKB_U262-161N-4BVC11 -> Connector_USB:USB_C_Receptacle_HRO_TYPE-C-31-M-12; symbol mainboard-rescue:USB_C_Receptacle_USB2.0-Connector -> Connector:USB_C_Receptacle_USB2.0_16P
- J4: renamed from J18; footprint mainboard:SCREWTERMINAL-3.5MM-2_LOCK -> mainboard:PHOENIX_1985807; symbol mainboard:M023.5MM_LOCK -> Connector_Generic:Conn_01x02
- J5: renamed from J16; footprint mainboard:SCREWTERMINAL-3.5MM-2_LOCK -> mainboard:PHOENIX_1985807; symbol mainboard:M023.5MM_LOCK -> Connector_Generic:Conn_01x02
- J6: renamed from J17; footprint mainboard:SCREWTERMINAL-3.5MM-2_LOCK -> mainboard:PHOENIX_1985807; symbol mainboard:M023.5MM_LOCK -> Connector_Generic:Conn_01x02
- J7: renamed from J28; footprint mainboard:USB_C_Receptacle_XKB_U262-161N-4BVC11 -> Connector_USB:USB_C_Receptacle_HRO_TYPE-C-31-M-12; symbol mainboard-rescue:USB_C_Receptacle_USB2.0-Connector -> Connector:USB_C_Receptacle_USB2.0_16P
- J8: renamed from J24; footprint (none) -> Connector_Card:microSD_HC_Molex_104031-0811
- J9: renamed from J1; footprint (none) -> Connector_PinHeader_1.27mm:PinHeader_2x05_P1.27mm_Vertical_SMD
- renumbered C29 to C26, C24 to C27, C31 to C28, C64 to C30, R144 to R56, R145 to R60, R146 to R65, U7 to U15, U10 to U16
Connections:
- net 3.3V: now also C31.1, C32.1
- net DBus1+: now also U15.6 (I/O1)
- net DBus1-: now also U15.4 (I/O2)
- net DBus2+: now also U16.6 (I/O1)
- net DBus2-: now also U16.4 (I/O2)
- net GND: now also C31.2, C32.2
- net GNDREF: now also J1.S1 (SHIELD), J2.2 (Pin_2), J2.4 (Pin_4)
- net VCHRG: now also J2.1 (Pin_1), J2.3 (Pin_3)
- removed net DN: U15.4 (I/O2), U16.4 (I/O2)
- removed net DP: U15.6 (I/O1), U16.6 (I/O1)
Other:
- note added: "USB-C Connector for RF MCU"

Commit message: v1.1 Schematic
Parts:
- added C50: 3.3nF, Capacitor_SMD:C_0603_1608Metric, symbol Device:C_Small
- added R26: 1K, Resistor_SMD:R_0603_1608Metric, symbol Device:R_Small
- added R8: ?R, Resistor_SMD:R_2512_6332Metric, symbol Device:R_Small
- added U9: ADM1176-1ARMZ-R7, Package_SO:MSOP-10_3x3mm_P0.5mm, symbol Mainboard:ADM1176-1ARMZ-R7
Connections:
- net GND: now also C50.1, U9.4 (GND)
- net VBATT: now also R8.2, U9.1 (VCC)
- new net: R26.2, U9.3 (ON)
- new net: C50.2, U9.5 (TIMER)
- new net PWR_SCL: U9.6 (SCL)
- new net PWR_SDA: U9.7 (SDA)
- new net VSYS: R26.1, R8.1, U9.2 (SENSE)
- no-connect marks 11 -> 14
Other:
- note added: "0x4A"
- note added: "Board Power Monitor"
- note added: "I2C1 ADDR"
