File: Bus_Protection.kicad_sch (KiCad schematic)
At the start: 83 parts, among them Q11 MMDT2907, Q12 BSS138DWQ-7, Q13 BSS138DWQ-7, Q15 MBT2222ADW1T1, Q16 MBT2222ADW1T1, Q17 BSS138DWQ-7, Q18 BSS138DWQ-7, Q19 BSS138DWQ-7, Q20 MBT2222ADW1T1, Q28 MBT2222ADW1T1, Q29 BSS138DWQ-7, Q30 MBT2222ADW1T1, Q4 BSS138DWQ-7, Q5 MBT2222ADW1T1, Q6 BSS138DWQ-7, Q7 MBT2222ADW1T1, Q8 MBT2222ADW1T1

Commit message: Complete layout
Parts:
- removed C55, C56: 10nF, Capacitor_SMD:C_0603_1608Metric, symbol Device:C
- removed Q11: MMDT2907, Package_TO_SOT_SMD:SOT-363_SC-70-6, symbol mainboard:MMDT2907
- removed Q17, Q29: BSS138DWQ-7, mainboard:BSS138DWQ-7, symbol mainboard:BSS138DWQ-7
- removed Q28, Q30: MBT2222ADW1T1, Package_TO_SOT_SMD:SOT-363_SC-70-6, symbol Transistor_BJT:MBT2222ADW1T1
- removed R119, R124: 200K, Resistor_SMD:R_0603_1608Metric, symbol Device:R_Small
- removed R120, R48: 100K, Resistor_SMD:R_0603_1608Metric, symbol Device:R_Small
- removed R121, R60: 680R, Resistor_SMD:R_0603_1608Metric, symbol Device:R_Small
- removed R122, R123, R77, R78: 10K, Resistor_SMD:R_0603_1608Metric, symbol Device:R_Small
- removed R125, R126: 0R, Resistor_SMD:R_0603_1608Metric, symbol Device:R_Small
- added Q16, Q17: MMBT2907, Package_TO_SOT_SMD:SOT-23, symbol Mainboard:MMBT2907
- Q11: renamed from Q19; footprint mainboard:BSS138DWQ-7 -> Package_TO_SOT_SMD:SOT-363_SC-70-6; symbol mainboard:BSS138DWQ-7 -> Mainboard:BSS138DWQ-7
- Q13: renamed from Q4; footprint mainboard:BSS138DWQ-7 -> Package_TO_SOT_SMD:SOT-363_SC-70-6; symbol mainboard:BSS138DWQ-7 -> Mainboard:BSS138DWQ-7
- Q15: renamed from Q6; footprint mainboard:BSS138DWQ-7 -> Package_TO_SOT_SMD:SOT-363_SC-70-6; symbol mainboard:BSS138DWQ-7 -> Mainboard:BSS138DWQ-7
- Q5: renamed from Q12; footprint mainboard:BSS138DWQ-7 -> Package_TO_SOT_SMD:SOT-363_SC-70-6; symbol mainboard:BSS138DWQ-7 -> Mainboard:BSS138DWQ-7
- Q7: renamed from Q13; footprint mainboard:BSS138DWQ-7 -> Package_TO_SOT_SMD:SOT-363_SC-70-6; symbol mainboard:BSS138DWQ-7 -> Mainboard:BSS138DWQ-7
- Q9: renamed from Q18; footprint mainboard:BSS138DWQ-7 -> Package_TO_SOT_SMD:SOT-363_SC-70-6; symbol mainboard:BSS138DWQ-7 -> Mainboard:BSS138DWQ-7
- renumbered C8 to C40, C40 to C41, C41 to C42, C42 to C43, C46 to C44, C48 to C45, Q16 to Q10, Q5 to Q12, Q20 to Q14, Q7 to Q4, Q8 to Q6, Q15 to Q8, R108 to R23, R109 to R44, R117 to R45, R118 to R48, R101 to R50, R104 to R54
Connections:
- net MISO: now also Q16.3 (C), Q17.3 (C)
- net SCL1: no longer Q12.1 (E1), Q12.3 (C2), R45.2
- net SDA1: no longer Q14.1 (E1), Q14.3 (C2), R48.2
- net at R68.1: now also Q17.1 (B)
- net at R99.1: now also Q17.2 (E)
- net at R53.1: now also Q16.2 (E)
- net at R92.1: now also Q16.1 (B)
- new net SCL3: Q12.1 (E1), Q12.3 (C2), R45.2
- new net SDA3: Q14.1 (E1), Q14.3 (C2), R48.2
Other:
- note removed: "I2C Bus Protection - Jetson Power"
- moved on the sheet: R97, R98

Commit message: v1 Final
Other:
- note added: "SPI Bus Protection - UHF Radio MCU"
- note removed: "SPI Bus Protection - UHF Radio"
Changed lines of the file:
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@@
 		)
 	)
-	(text "SPI Bus Protection - UHF Radio"
+	(text "SPI Bus Protection - UHF Radio MCU"
 		(exclude_from_sim no)
-		(at 215.9 60.96 0)
+		(at 212.09 60.96 0)
 		(effects
 			(font

Commit message: Stash
Parts:
- R23, R44, R45, R48, R50, R54, R97, R98: value 0R -> DNI (0R)
Connections:
- net SCL3 renamed SCL2
- net SDA3 renamed SDA2
Changed lines of the file:
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@@
 		)
 	)
-	(global_label "SCL3"
+	(global_label "SCL2"
 		(shape bidirectional)
 		(at 91.44 177.8 180)
@@
 		)
 	)
-	(global_label "SCL3"
+	(global_label "SCL2"
 		(shape bidirectional)
 		(at 123.19 43.18 180)
@@
 		)
 	)
-	(global_label "SDA3"
+	(global_label "SDA2"
 		(shape bidirectional)
 		(at 165.1 43.18 180)
@@
 		)
 	)
-	(global_label "SDA3"
+	(global_label "SDA2"
 		(shape bidirectional)
 		(at 91.44 181.61 180)
@@
 			)
 		)
-		(property "Value" "0R"
-			(at 57.912 190.5 90)
+		(property "Value" "DNI (0R)"
+			(at 60.96 190.754 90)
 			(effects
 				(font
@@
 		)
 		(property "DNI" "DNI"
-			(at 54.61 193.548 90)
+			(at 54.61 191.77 90)
 			(effects
 				(font
@@
 			)
 		)
-		(property "Value" "0R"
-			(at 57.912 176.53 90)
+		(property "Value" "DNI (0R)"
+			(at 60.706 176.53 90)
 			(effects
 				(font
@@
 		)
 		(property "DNI" "DNI"
-			(at 54.61 176.022 90)
+			(at 54.61 177.8 90)
 			(effects
 				(font
@@
 			)
 		)
-		(property "Value" "0R"
-			(at 57.912 180.34 90)
+		(property "Value" "DNI (0R)"
+			(at 60.706 180.34 90)
 			(effects
 				(font
@@
 		)
 		(property "DNI" "DNI"
-			(at 54.61 183.388 90)
+			(at 54.61 181.61 90)
 			(effects
 				(font
@@
 			)
 		)
-		(property "Value" "0R"
-			(at 140.462 180.34 90)
+		(property "Value" "DNI (0R)"
+			(at 143.51 180.34 90)
 			(effects
 				(font
@@
 		)
 		(property "DNI" "DNI"
-			(at 137.16 183.388 90)
+			(at 137.16 181.61 90)
 			(effects
 				(font
@@
 			)
 		)
-		(property "Value" "0R"
-			(at 140.462 186.69 90)
+		(property "Value" "DNI (0R)"
+			(at 143.51 186.69 90)
 			(effects
 				(font
@@
 		)
 		(property "DNI" "DNI"
-			(at 137.16 189.738 90)
+			(at 137.16 187.96 90)
 			(effects
 				(font
@@
 			)
 		)
-		(property "Value" "0R"
-			(at 57.912 186.69 90)
+		(property "Value" "DNI (0R)"
+			(at 60.96 186.69 90)
 			(effects
 				(font
@@
 		)
 		(property "DNI" "DNI"
-			(at 54.61 186.182 90)
+			(at 54.61 187.96 90)
 			(effects
 				(font
@@
 			)
 		)
-		(property "Value" "0R"
-			(at 99.822 180.34 90)
+		(property "Value" "DNI (0R)"
+			(at 102.87 180.34 90)
 			(effects
 				(font
@@
 		)
 		(property "DNI" "DNI"
-			(at 96.52 183.388 90)
+			(at 96.52 181.61 90)
 			(effects
 				(font
@@
 			)
 		)
-		(property "Value" "0R"
-			(at 99.822 176.53 90)
+		(property "Value" "DNI (0R)"
+			(at 102.87 176.53 90)
 			(effects
 				(font
@@
 		)
 		(property "DNI" "DNI"
-			(at 96.52 176.022 90)
+			(at 96.52 177.8 90)
 			(effects
 				(font
