File: Mainboard.kicad_pcb (KiCad board)
At the start: 4 copper layers, 90.2 x 95.9 mm, 265 parts, among them J1 USB_C_Receptacle_USB2.0, J10 200528-0100, J11 200528-0100, J12 200528-0100, J13 200528-0100, J14 200528-0100, J15 200528-0100, J16 200528-0100, J17 200528-0100, J18 200528-0100, J19 Conn_01x09, J2 282834-4, J20 Conn_01x04, J21 Conn_01x06, J22 U.FL-R-SMT-1, J23 U.FL-R-SMT-1, J24 Conn_02x05_Odd_Even, J3 282834-4, J4 1985807, J5 1985807, J6 1985807, J7 USB_C_Receptacle_USB2.0, J8 Micro_SD_Card_Det2, J9 Conn_02x05_Odd_Even, Q1 IRLML2803, Q10 MBT2222ADW1T1, Q11 BSS138DWQ-7, Q12 MBT2222ADW1T1, Q13 BSS138DWQ-7, Q14 MBT2222ADW1T1, Q15 BSS138DWQ-7, Q16 MMBT2907, Q17 MMBT2907, Q18 IRLML2803, Q19 IRF7404, Q2 MBT2222ADW1T1, Q21 IRLML2803, Q22 IRLML2803, Q23 IRF7404, Q3 MBT2222ADW1T1, Q4 MBT2222ADW1T1, Q5 BSS138DWQ-7, Q6 MBT2222ADW1T1, Q7 BSS138DWQ-7, Q8 MBT2222ADW1T1, Q9 BSS138DWQ-7, SW1 KMR231NG LFS, SW2 KMR231NG LFS, SW3 KMR231NG LFS, U1 MAX706RESA+, U10 MR25H40MDF, U11 MAX706RESA+, U12 E22-900M30S, U13 S1216V8, U14 EP2W+, U15 USBLC6-2SC6, U16 USBLC6-2SC6, U17 RP2040, U2 ATSAMD51J20A-AU, U3 BMX160, U4 DS3231S, U5 MR25H40MDF, U6 TPS7A4501DCQT, U7 TPS54226PWPR, U8 BQ25883RGER, U9 ADM1176-1ARMZ-R7, Y1 32.768kHz, Y2 ABM8-272-T3

Commit message: v1.1 Layout
Parts:
- removed C3: 0.1uF, Capacitor_SMD:C_0603_1608Metric
- removed R1: 316K, Resistor_SMD:R_0603_1608Metric
- removed R102, R103: 0R, Resistor_SMD:R_0603_1608Metric
- removed R2: 110K, Resistor_SMD:R_0603_1608Metric
- R20, R21, R22, R5: moved to B.Cu
- moved D2 79.1 mm to (154.8, 145.1)
- moved C55 79.1 mm to (154.8, 140.7)
- moved R105 66.9 mm to (161.0, 138.0)
- moved SW3 62.3 mm to (167.4, 137.3)
- moved D4 60.0 mm to (163.3, 137.3), turned to -90 degrees
- moved R22 59.0 mm to (152.5, 116.9), turned to 180 degrees
- moved R21 57.7 mm to (152.5, 119.4), turned to 180 degrees
- moved J24 54.2 mm to (176.9, 135.5)
- moved R104 52.8 mm to (161.0, 136.5), turned to 180 degrees
- moved C71 48.1 mm to (161.0, 119.8), turned to 180 degrees
- moved C56 42.5 mm to (163.4, 115.7)
- moved R9 40.8 mm to (170.7, 118.3), turned to 180 degrees
- moved C63 39.6 mm to (166.2, 120.6), turned to 90 degrees
- moved SW2 34.9 mm to (167.4, 115.7)
- moved U11 33.6 mm to (176.0, 120.5), turned to 180 degrees
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Connections:
- net Net-(U17-USB_DM) renamed /RF and GPS/D2-
- net Net-(U17-USB_DP) renamed /RF and GPS/D2+
- U17 pad 11: RF_RST -> unconnected-(U17-GPIO8-Pad11)
- U17 pad 12: RF_BUSY -> unconnected-(U17-GPIO9-Pad12)
- U17 pad 18: RF_IO2 -> RF_RST
- U17 pad 27: RF_TXEN -> RF_BUSY
- U17 pad 28: RF_RXEN -> RF_WDT_WDI
- U17 pad 30: Net-(U17-GPIO19) -> UHF_MOSI
- U17 pad 31: Net-(U17-GPIO20) -> UHF_MISO
- U17 pad 36: RF_WDT_WDI -> unconnected-(U17-GPIO24-Pad36)
- U17 pad 37: /RF and GPS/RF_NEOPIXEL -> RF_IO2
- U17 pad 4: unconnected-(U17-GPIO2-Pad4) -> /RF and GPS/RF_NEOPIXEL
- U17 pad 6: unconnected-(U17-GPIO4-Pad6) -> RF_RXEN
- U17 pad 8: unconnected-(U17-GPIO6-Pad8) -> RF_TXEN
- U2 pad 16: Net-(U2-PA07) -> unconnected-(U2-PA07-Pad16)
Routing:
- net RF_3.3V: track 0.00 -> 21.6 mm, vias 0 -> 2
- net ~{RF_RST}: track 18.5 -> 37.8 mm, vias 0 -> 3
- net GND: track 60.4 -> 76.6 mm, vias 224 -> 259
- net /RF and GPS/RF_NEOPIXEL: track 10.7 -> 24.6 mm, vias 1 -> 2
- net RF_TXEN: track 11.7 -> 25.0 mm, vias 1 -> 2
- net SCK: track 87.5 -> 100.4 mm
- net RF_CS: track 6.09 -> 18.3 mm, vias 0 -> 1
- net RF_RXEN: track 10.3 -> 22.2 mm, vias 1 -> 2
- net RF_SCK: track 6.15 -> 17.5 mm, vias 0 -> 1
- net Net-(U17-XIN): track 0.00 -> 11.3 mm
- net UHF_MISO: track 5.14 -> 16.4 mm, vias 1 -> 2
- net MISO: track 87.7 -> 77.3 mm
- net /RF and GPS/QSPI_D3: track 6.62 -> 16.8 mm
- net /Avionics/NEOPIXEL: track 43.5 -> 53.0 mm, vias 2 -> 3
- net /RF and GPS/QSPI_SCK: track 5.02 -> 14.5 mm
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- added copper zone on F.Cu, net RF_3.3VA
Other:
- board text added: "BOOTSEL"
- board text added: "RESET"
- board text added: "mainboard.v1.1"
- board text removed: "mainboard.v1"

Commit message: Stash
Parts:
- added R1: 0R, Resistor_SMD:R_0603_1608Metric, F.Cu at (168.8, 133.1)
- added R2: 0R, Resistor_SMD:R_0603_1608Metric, F.Cu at (170.2, 133.1)
- R23, R44, R45, R48, R50, R54, R97, R98: value 0R -> DNI (0R)
- moved REF** 1.12 mm to (129.3, 128.3)
- moved C65 1.09 mm to (167.3, 133.1)
Connections:
- J17 pad 10: SCL3 -> SCL2
- J17 pad 9: SDA3 -> SDA2
- J18 pad 10: SCL3 -> SCL2
- J18 pad 9: SDA3 -> SDA2
- Q12 pad 1: SCL3 -> SCL2
- Q12 pad 3: SCL3 -> SCL2
- Q14 pad 1: SDA3 -> SDA2
- Q14 pad 3: SDA3 -> SDA2
- R45 pad 2: SCL3 -> SCL2
- R48 pad 2: SDA3 -> SDA2
- U17 pad 11: unconnected-(U17-GPIO8-Pad11) -> /RF and GPS/TX1
- U17 pad 12: unconnected-(U17-GPIO9-Pad12) -> /RF and GPS/RX1
- U17 pad 34: unconnected-(U17-GPIO22-Pad34) -> RF_IO2
- U17 pad 35: RF_WDT_EN -> unconnected-(U17-GPIO23-Pad35)
- U17 pad 37: RF_IO2 -> RF_WDT_EN
- U2 pad 35: SDA3 -> UHF_TX
- U2 pad 36: SCL3 -> UHF_RX
Routing:
- net SDA3: track 139.5 -> 0.00 mm, vias 6 -> 0
- net SCL3: track 128.4 -> 0.00 mm, vias 5 -> 0
- net SDA2: track 127.6 -> 231.6 mm, vias 4 -> 9
- net SCL2: track 124.2 -> 219.9 mm, vias 4 -> 8
- net UHF_TX: track 0.00 -> 55.4 mm, vias 0 -> 2
- net UHF_RX: track 0.00 -> 55.1 mm, vias 0 -> 2
- net /RF and GPS/RX1: track 0.00 -> 2.45 mm
- net /RF and GPS/TX1: track 0.00 -> 2.01 mm
- net RF_IO2: track 18.4 -> 20.1 mm
- net RF_WDT_EN: track 12.0 -> 13.4 mm
Other:
- board text added: "ARGUS-1 Cubesat Carnegie Mellon University Mainboard v1.1"
- board text removed: "ARGUS-1 Cubesat Carnegie Mellon University Mainboard v1"
- board text removed: "SCL3"
- board text removed: "SDA3"
