File: RF_and_GPS.kicad_sch (KiCad schematic)
At the start: 34 parts, among them J12 U.FL-R-SMT-1, J2 U.FL-R-SMT-1, J29 Conn_02x05_Odd_Even, J7 U.FL-R-SMT-1, Q21 IRF7404, Q38 IRLML2803, Q9 IRLML2803, SW2 KMR231NG LFS, U11 MAX706RESA+, U13 EP2W+, U14 S1216V8, U23 RFM98PW, U9 ATSAMD21E18A-A

Commit message: Complete layout
Parts:
- removed C44: 10uF, symbol Device:C_Small
- removed J2: U.FL-R-SMT-1, symbol Connector:Conn_Coaxial_Small
- removed JP10: SolderJumper_2_Open, symbol Jumper:SolderJumper_2_Open
- added C58, C59: 8pF, Capacitor_SMD:C_0603_1608Metric, symbol Device:C_Small
- added Q18: IRLML2803, Package_TO_SOT_SMD:SOT-23, symbol Mainboard:IRLML2803
- added Q19: IRF7404, Package_SO:SOIC-8_3.9x4.9mm_P1.27mm, symbol Mainboard:IRF7404
- added R10, R11, R20, R21, R22, R9: 10K, Resistor_SMD:R_0603_1608Metric, symbol Device:R_Small
- added R16: 4.7K, Resistor_SMD:R_0603_1608Metric, symbol Device:R_Small
- added R18: 3.3K, Resistor_SMD:R_0603_1608Metric, symbol Device:R_Small
- added Y2: 32.768kHz, Crystal:Crystal_SMD_3215-2Pin_3.2x1.5mm, symbol Device:Crystal_Small
- C51: renamed from C75; footprint (none) -> Capacitor_SMD:C_0603_1608Metric
- C52: renamed from C66; footprint (none) -> Capacitor_SMD:C_0603_1608Metric
- C53: renamed from C67; footprint (none) -> Capacitor_SMD:C_0603_1608Metric
- C54: renamed from C71; footprint (none) -> Capacitor_SMD:C_0603_1608Metric
- C55: renamed from C80; symbol mainboard:C_Small -> Device:C_Small
- C56: renamed from C76; symbol mainboard:C_Small -> Device:C_Small
- J22: renamed from J7; footprint (none) -> Connector_Coaxial:U.FL_Hirose_U.FL-R-SMT-1_Vertical
- J23: renamed from J12; footprint (none) -> Connector_Coaxial:U.FL_Hirose_U.FL-R-SMT-1_Vertical
- J24: renamed from J29; footprint (none) -> Connector_PinHeader_1.27mm:PinHeader_2x05_P1.27mm_Vertical_SMD
- Q1: renamed from Q38; symbol Transistor_FET:IRLML2060 -> Mainboard:IRLML2803
- Q22: renamed from Q9; symbol Transistor_FET:IRLML2060 -> Mainboard:IRLML2803
- Q23: renamed from Q21; footprint mainboard:NDS8434 -> Package_SO:SOIC-8_3.9x4.9mm_P1.27mm; symbol mainboard:NDS8434 -> Mainboard:IRF7404
- R88: renamed from R156; footprint (none) -> Resistor_SMD:R_0603_1608Metric
- R91: renamed from R137; footprint (none) -> Resistor_SMD:R_0603_1608Metric
- SW2: footprint mainboard:BTN_KMR2_4.6X2.8 -> Button_Switch_SMD:SW_Push_1P1T_NO_CK_KMR2; symbol mainboard:SWITCH_SMT4.6X2.8 -> Mainboard:KMR231
- U11: symbol mainboard:MAX708RESA+ -> Mainboard:MAX706RESA+
- U12: renamed from U23; value RFM98PW -> E22-900M30S; footprint mainboard:RFM95PW -> mainboard:XCVR_E22-900M30S; symbol mainboard:RFM98PW -> Mainboard:E22-900M30S
- U13: renamed from U14; symbol mainboard:S1216V8 -> Mainboard:S1216V8
- U14: renamed from U13; footprint mainboard:QFN32-5X5MM -> mainboard:EP2W+; symbol mainboard:EP2W+ -> Mainboard:EP2W+
- renumbered C79 to C57, D4 to D2, R149 to R78, R150 to R79, R151 to R80, R152 to R81, U9 to U10
Connections:
- net RF_ANT is gone; now on net GND: U12.1 (GND)
- net 3.3V: now also Q19.1 (Source), Q19.2 (Source), Q19.3 (Source), R18.1; no longer C55.1, D2.1 (VDD)
- net GND: now also SW2.2 (S1), U12.11 (GND), U12.12 (GND), U12.20 (GND), U12.22 (GND), U12.3 (GND), U12.4 (GND), U12.5 (GND), C58.2, C59.2, Q18.2 (S), R11.2, R21.2, R22.2, R9.2; no longer SW2.B (S), SW2.B' (S1), U12.16 (GND), U12.17 (GND)
- net RF_3.3V: now also C55.1, D2.1 (VDD), Q19.5 (Drain), Q19.6 (Drain), Q19.7 (Drain), Q19.8 (Drain), R10.1, R20.1
- net RF_CS: now also U12.19 (NSS); no longer U12.13 (NSS)
- net RF_MISO: now also U12.16 (MISO); no longer U12.10 (MISO)
- net RF_MOSI: now also U12.17 (MOSI); no longer U12.11 (MOSI)
- net RF_RST: now also U10.3 (PA02), U12.15 (nRST), R20.2; no longer U10.2 (PA01), U12.14 (RESET)
- net RF_SCK: now also U12.18 (SCK); no longer U12.12 (SCK)
- net RF_VDD: now also U12.10 (VCC), U12.9 (VCC); no longer U12.5 (VCC)
- net SAMD21_NEOPIXEL: now also U10.20 (PA19); no longer U10.1 (PA00)
- net SAMD21_SWC: now also R10.2
- net SAMD21_WDT_EN: now also U10.21 (PA22)
- net SAMD21_WDT_WDI: now also U10.22 (PA23), R9.1
- net ~{SAMD21_RST}: now also SW2.1 (P1); no longer SW2.A (P), SW2.A' (P1)
- net RF_TXEN: now reaches U12.7 (TXEN)
- net RF_TXEN: now also U10.17 (PA16), R22.1
- net RF_IO2: now reaches U12.8 (DIO2)
- net RF_IO2: now also U10.16 (PA15)
- net RF_IO1: now reaches U10.15 (PA14)
- net RF_IO1: now also U12.13 (DIO1)
- net RF_RXEN: now reaches U10.18 (PA17)
- net RF_RXEN: now also U12.6 (RXEN), R21.1
- removed net RF_IO0: U10.3 (PA02), U12.6 (GPIO_0)
- net RF_IO4 renamed RF_BUSY
- net RF_BUSY: now also U12.14 (BUSY); no longer U12.4 (GPIO_4)
- new net: C58.1, U10.1 (PA00), Y2.1
- new net: Q18.3 (D), Q19.4 (Gate), R18.2
- new net: C59.1, U10.2 (PA01), Y2.2
- new net: Q18.1 (G), R16.2
- new net UHF_EN: R11.1, R16.1
- no-connect marks 33 -> 23
Other:
- note added: "UHF 3.3V"
- moved on the sheet: C51, C55, C57, D2, J24, Q1, Q22, R12, R17, R19, R5, R79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

Commit message: v1 Final
Other:
- note added: "SPI 1 Mainboard (Master) RF MCU (Slave)"
- note added: "SPI 2 RF MCU (Master) RF Module(Slave)"
Changed lines of the file:
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@@
+		)
+	)
+	(polyline
+		(pts
+			(xy 51.054 51.308) (xy 48.768 51.308)
+		)
+		(stroke
+			(width 0)
+			(type dash)
 		)
 	)
@@
 		)
 	)
+	(polyline
+		(pts
+			(xy 48.768 51.308) (xy 48.768 62.23)
+		)
+		(stroke
+			(width 0)
+			(type dash)
+		)
+	)
 	(wire
 		(pts
@@
 		)
 	)
+	(polyline
+		(pts
+			(xy 48.768 62.23) (xy 48.768 73.152)
+		)
+		(stroke
+			(width 0)
+			(type dash)
+		)
+	)
 	(wire
 		(pts
@@
 		)
 	)
+	(polyline
+		(pts
+			(xy 48.768 62.23) (xy 51.308 62.23)
+		)
+		(stroke
+			(width 0)
+			(type dash)
+		)
+	)
 	(wire
 		(pts
@@
 		)
 	)
+	(polyline
+		(pts
+			(xy 51.054 62.23) (xy 48.768 62.23)
+		)
+		(stroke
+			(width 0)
+			(type dash)
+		)
+	)
 	(wire
 		(pts
@@
 			(width 0)
 			(type default)
+		)
+	)
+	(polyline
+		(pts
+			(xy 48.768 73.152) (xy 51.308 73.152)
+		)
+		(stroke
+			(width 0)
+			(type dash)
 		)
 	)
@@
 		)
 	)
+	(text "SPI 2\nRF MCU (Master)\nRF Module(Slave)"
+		(exclude_from_sim no)
+		(at 37.846 56.388 0)
+		(effects
+			(font
+				(size 1.27 1.27)
+			)
+		)
+	)
 	(text "SWD Connector"
 		(exclude_from_sim no)
@@
 		)
 	)
+	(text "SPI 1\nMainboard (Master)\nRF MCU (Slave)"
+		(exclude_from_sim no)
+		(at 37.846 67.31 0)
+		(effects
+			(font
+				(size 1.27 1.27)
+			)
+		)
+	)

Commit message: v1.1 Schematic
Parts:
- removed Q18, Q22: IRLML2803, Package_TO_SOT_SMD:SOT-23, symbol Mainboard:IRLML2803
- removed Q19, Q23: IRF7404, Package_SO:SOIC-8_3.9x4.9mm_P1.27mm, symbol Mainboard:IRF7404
- removed R11, R12: 10K, Resistor_SMD:R_0603_1608Metric, symbol Device:R_Small
- removed R16, R17: 4.7K, Resistor_SMD:R_0603_1608Metric, symbol Device:R_Small
- removed R18, R19: 3.3K, Resistor_SMD:R_0603_1608Metric, symbol Device:R_Small
- removed U10: ATSAMD21E18A-A, Package_QFP:TQFP-32_7x7mm_P0.8mm, symbol MCU_Microchip_SAMD:ATSAMD21E18A-A
- removed Y2: 32.768kHz, Crystal:Crystal_SMD_3215-2Pin_3.2x1.5mm, symbol Device:Crystal_Small
- added C61, C62, C63, C64, C65, C66, C69, C70: 0.1uF, Capacitor_SMD:C_0603_1608Metric, symbol Device:C_Small
- added C67, C68: 10uF, Capacitor_SMD:C_0603_1608Metric, symbol Device:C_Small
- added C71: 1uF, Capacitor_SMD:C_0603_1608Metric, symbol Device:C_Small
- added D4: GREEN LED, LED_SMD:LED_0603_1608Metric, symbol Device:LED_Small
- added FB2: FerriteBead_Small, Inductor_SMD:L_0603_1608Metric, symbol Device:FerriteBead_Small
- added R100, R101: 27R, Resistor_SMD:R_0603_1608Metric, symbol Device:R_Small
- added R102, R103: 0R, Resistor_SMD:R_0603_1608Metric, symbol Device:R_Small
- added R104: 10K, Resistor_SMD:R_0603_1608Metric, symbol Device:R_Small
- added R105: 1K, Resistor_SMD:R_0603_1608Metric, symbol Device:R_Small
- added SW3: KMR231NG LFS, Button_Switch_SMD:SW_Push_1P1T_NO_CK_KMR2, symbol Mainboard:KMR231
- added U10: MR25H40MDF, Package_DFN_QFN:DFN-8-1EP_6x5mm_P1.27mm_EP2x2mm, symbol Mainboard:MR25H40MDF
- added U17: RP2040, Package_DFN_QFN:QFN-56-1EP_7x7mm_P0.4mm_EP3.2x3.2mm, symbol MCU_RaspberryPi:RP2040
- added Y2: ABM8-272-T3, Crystal:Crystal_SMD_3225-4Pin_3.2x2.5mm, symbol Device:Crystal_GND24_Small
- C54: value 10uF -> 0.1uF
- C58, C59: value 8pF -> 15pF
- R10: value 10K -> 1K
Connections:
- net GND: now also C61.2, C62.2, C63.2, C64.2, C65.2, C66.2, C67.2, C68.2, C69.2, C70.2, C71.2, SW3.2 (S1), U10.4 (VSS), U10.9 (EP), U17.19 (TESTEN), U17.57 (GND), Y2.2, Y2.4
- net RF_3.3V: now also C61.1, C62.1, C63.1, C64.1, C65.1, C66.1, C67.1, C70.1, C71.1, FB2.1, R104.2, U10.8 (VDD), U17.1 (IOVDD), U17.10 (IOVDD), U17.22 (IOVDD), U17.33 (IOVDD), U17.42 (IOVDD), U17.44 (VREG_IN), U17.48 (USB_VDD), U17.49 (IOVDD); no longer C52.1, C53.1, R10.1
- net RF_BUSY: now also U17.12 (GPIO9)
- net RF_CS: now also U17.16 (GPIO13)
- net RF_IO1: now also U17.17 (GPIO14)
- net RF_IO2: now also U17.18 (GPIO15)
- net RF_MISO: now also U17.15 (GPIO12)
- net RF_MOSI: now also U17.14 (GPIO11)
- net RF_RST: now also U17.11 (GPIO8)
- net RF_RXEN: now also U17.28 (GPIO17)
- net RF_SCK: now also U17.13 (GPIO10)
- net RF_TXEN: now also U17.27 (GPIO16)
- net UHF_CS: now also U17.32 (GPIO21)
- net UHF_MISO: now also R103.2
- net UHF_MOSI: now also R102.2
- net UHF_SCK: now also U17.29 (GPIO18)
- net USB_D2+: now also R100.1
- net USB_D2-: now also R101.2
- net at C58.1: now also U17.20 (XIN), Y2.1
- net at C59.1: now also R10.2, Y2.3
- net +1V2: now reaches C51.1
- net +1V2: now also C52.1, C53.1, U17.23 (DVDD), U17.45 (VREG_VOUT), U17.50 (DVDD)
- net SAMD21_NEOPIXEL renamed RF_NEOPIXEL
- net RF_NEOPIXEL: now also U17.37 (GPIO25)
- net SAMD21_SWC renamed RF_SWC
- net RF_SWC: now also U17.24 (SWCLK); no longer R10.2
- net SAMD21_SWD renamed RF_SWD
- net RF_SWD: now also U17.25 (SWD)
- net SAMD21_WDT_EN renamed RF_WDT_EN
- net RF_WDT_EN: now also U17.35 (GPIO23)
- net SAMD21_WDT_WDI renamed RF_WDT_WDI
- net RF_WDT_WDI: now also U17.36 (GPIO24)
- net ~{SAMD21_RST} renamed ~{RF_RST}
- net ~{RF_RST}: now also U17.26 (RUN)
- new net: R10.1, U17.21 (XOUT)
- new net: D4.1 (K), SW3.1 (P1)
- new net: R102.1, U17.30 (GPIO19)
- new net: R101.1, U17.46 (USB_DM)
- new net: D4.2 (A), R105.2
- new net: R100.2, U17.47 (USB_DP)
- new net: R103.1, U17.31 (GPIO20)
- new net QSPI_D0: U10.5 (SI), U17.53 (QSPI_SD0)
- new net QSPI_D1: U10.2 (SO), U17.55 (QSPI_SD1)
- new net QSPI_D2: U10.3 (~{WP}), U17.54 (QSPI_SD2)
- new net QSPI_D3: U10.7 (~{HOLD}), U17.51 (QSPI_SD3)
- new net QSPI_SCK: U10.6 (SCK), U17.52 (QSPI_SCLK)
- new net QSPI_SS: R104.1, R105.1, U10.1 (~{CS}), U17.56 (QSPI_SS)
- new net RF_3.3VA: C68.1, C69.1, FB2.2, U17.43 (ADC_AVDD)
- no-connect marks 23 -> 33
Other:
- note added: "BOOTSEL"
- note added: "DECOUPLING"
- note added: "MRAM - Nonvolatile Memory (4MB storage)"
- note added: "PWM4 A"
- note added: "SPI 0 Mainboard (Master) RF MCU (Slave)"
- note added: "SPI 1 RF MCU (Master) RF Module (Slave)"
- note removed: "GPS Power"
- note removed: "SPI 1 Mainboard (Master) RF MCU (Slave)"
- note removed: "SPI 2 RF MCU (Master) RF Module(Slave)"
- note removed: "UHF 3.3V"
- moved on the sheet: C51, C52, C53, C55, C56, C57, C58, C59, D2, J22, J23, J24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

Commit message: v1.1 Layout
Parts:
- removed R102, R103: 0R, Resistor_SMD:R_0603_1608Metric, symbol Device:R_Small
Connections:
- net RF_BUSY: now also U17.27 (GPIO16); no longer U17.12 (GPIO9)
- net RF_IO2: now also U17.37 (GPIO25); no longer U17.18 (GPIO15)
- net RF_NEOPIXEL: now also U17.4 (GPIO2); no longer U17.37 (GPIO25)
- net RF_RST: now also U17.18 (GPIO15); no longer U17.11 (GPIO8)
- net RF_RXEN: now also U17.6 (GPIO4); no longer U17.28 (GPIO17)
- net RF_TXEN: now also U17.8 (GPIO6); no longer U17.27 (GPIO16)
- net RF_WDT_WDI: now also U17.28 (GPIO17); no longer U17.36 (GPIO24)
- net UHF_MISO: now also U17.31 (GPIO20)
- net UHF_MOSI: now also U17.30 (GPIO19)
- net D2-: now reaches R101.1, U17.46 (USB_DM)
- net D2+: now reaches R100.2, U17.47 (USB_DP)
Other:
- note removed: "PWM4 A"

Commit message: Stash
Parts:
- added R1, R2: 0R, Resistor_SMD:R_0603_1608Metric, symbol Device:R_Small
Connections:
- net RF_IO2: now also U17.34 (GPIO22); no longer U17.37 (GPIO25)
- net RF_WDT_EN: now also U17.37 (GPIO25); no longer U17.35 (GPIO23)
- net TX1: now reaches U17.11 (GPIO8)
- net TX1: now also R1.2
- net RX1: now reaches U17.12 (GPIO9)
- net RX1: now also R2.2
- new net UHF_RX: R1.1
- new net UHF_TX: R2.1
- no-connect marks 33 -> 31
Changed lines of the file:
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@@
 	)
 	(no_connect
-		(at 143.51 116.84)
+		(at 143.51 119.38)
 	)
 	(no_connect
@@
 	)
 	(no_connect
-		(at 143.51 83.82)
-	)
-	(no_connect
 		(at 228.6 135.89)
 	)
@@
 	)
 	(no_connect
-		(at 143.51 81.28)
-	)
-	(no_connect
 		(at 143.51 63.5)
 	)
@@
 	(wire
 		(pts
-			(xy 143.51 124.46) (xy 157.48 124.46)
-		)
-		(stroke
-			(width 0)
-			(type default)
-		)
-	)
-	(wire
-		(pts
 			(xy 203.2 86.36) (xy 193.04 86.36)
 		)
@@
 	(wire
 		(pts
+			(xy 143.51 81.28) (xy 148.59 81.28)
+		)
+		(stroke
+			(width 0)
+			(type default)
+		)
+	)
+	(wire
+		(pts
 			(xy 143.51 66.04) (xy 157.48 66.04)
 		)
@@
 	(wire
 		(pts
-			(xy 143.51 119.38) (xy 157.48 119.38)
-		)
-		(stroke
-			(width 0)
-			(type default)
-		)
-	)
-	(wire
-		(pts
 			(xy 67.31 26.67) (xy 67.31 27.94)
 		)
@@
 	(wire
 		(pts
+			(xy 143.51 83.82) (xy 148.59 83.82)
+		)
+		(stroke
+			(width 0)
+			(type default)
+		)
+	)
+	(wire
+		(pts
 			(xy 107.95 34.29) (xy 97.79 34.29)
 		)
@@
 	(wire
 		(pts
+			(xy 153.67 83.82) (xy 157.48 83.82)
+		)
+		(stroke
+			(width 0)
+			(type default)
+		)
+	)
+	(wire
+		(pts
 			(xy 107.95 26.67) (xy 120.65 26.67)
 		)
@@
 	(wire
 		(pts
+			(xy 153.67 81.28) (xy 157.48 81.28)
+		)
+		(stroke
+			(width 0)
+			(type default)
+		)
+	)
+	(wire
+		(pts
 			(xy 250.19 30.48) (xy 250.19 33.02)
 		)
@@
 	(wire
 		(pts
+			(xy 143.51 124.46) (xy 157.48 124.46)
+		)
+		(stroke
+			(width 0)
+			(type default)
+		)
+	)
+	(wire
+		(pts
 			(xy 57.15 34.29) (xy 57.15 35.56)
 		)
@@
 	(wire
 		(pts
+			(xy 143.51 116.84) (xy 157.48 116.84)
+		)
+		(stroke
+			(width 0)
+			(type default)
+		)
+	)
+	(wire
+		(pts
 			(xy 97.79 182.88) (xy 115.57 182.88)
 		)
@@
 		)
 	)
+	(label "RX1"
+		(at 143.51 83.82 0)
+		(fields_autoplaced yes)
+		(effects
+			(font
+				(size 0.635 0.635)
+			)
+			(justify left bottom)
+		)
+	)
 	(label "QSPI_SCK"
 		(at 77.47 93.98 0)
@@
 		)
 	)
+	(label "TX1"
+		(at 143.51 81.28 0)
+		(fields_autoplaced yes)
+		(effects
+			(font
+				(size 0.635 0.635)
+			)
+			(justify left bottom)
+		)
+	)
 	(label "D2+"
 		(at 87.63 68.58 0)
@@
 	(global_label "RF_WDT_EN"
 		(shape bidirectional)
-		(at 157.48 119.38 0)
+		(at 157.48 124.46 0)
 		(fields_autoplaced yes)
 		(effects
@@
 		)
 		(property "Intersheetrefs" "${INTERSHEET_REFS}"
-			(at 171.2258 119.38 0)
+			(at 171.2258 124.46 0)
 			(effects
 				(font
@@
 		)
 	)
-	(global_label "RF_IO2"
+	(global_label "UHF_TX"
 		(shape bidirectional)
-		(at 157.48 124.46 0)
+		(at 157.48 83.82 0)
 		(effects
 			(font
@@
 		)
 		(property "Intersheetrefs" "${INTERSHEET_REFS}"
-			(at 157.48 124.46 0)
+			(at 157.48 83.82 0)
 			(effects
 				(font
 					(size 1.27 1.27)
 				)
-				(justify right)
 				(hide yes)
 			)
@@
 		)
 	)
+	(global_label "RF_IO2"
+		(shape bidirectional)
+		(at 157.48 116.84 0)
+		(effects
+			(font
+				(size 1.27 1.27)
+			)
+			(justify left)
+		)
+		(property "Intersheetrefs" "${INTERSHEET_REFS}"
+			(at 157.48 116.84 0)
+			(effects
+				(font
+					(size 1.27 1.27)
+				)
+				(justify right)
+				(hide yes)
+			)
+		)
+	)
 	(global_label "RF_SWC"
 		(shape bidirectional)
@@
 		)
 	)
+	(global_label "UHF_RX"
+		(shape bidirectional)
+		(at 157.48 81.28 0)
+		(effects
+			(font
+				(size 1.27 1.27)
+			)
+			(justify left)
+		)
+		(property "Intersheetrefs" "${INTERSHEET_REFS}"
+			(at 157.48 81.28 0)
+			(effects
+				(font
+					(size 1.27 1.27)
+				)
+				(hide yes)
+			)
+		)
+	)
 	(global_label "RF_SWC"
 		(shape bidirectional)
@@
 	(symbol
 		(lib_id "Device:R_Small")
+		(at 151.13 81.28 270)
+		(unit 1)
+		(exclude_from_sim no)
+		(in_bom yes)
+		(on_board yes)
+		(dnp no)
+		(property "Reference" "R1"
+			(at 147.32 80.264 90)
+			(effects
+				(font
+					(size 1.27 1.27)
+				)
+			)
+		)
+		(property "Value" "0R"
+			(at 154.432 80.264 90)
+			(effects
+				(font
+					(size 1.27 1.27)
+				)
+			)
+		)
+		(property "Footprint" "Resistor_SMD:R_0603_1608Metric"
+			(at 151.13 81.28 0)
+			(effects
+				(font
+					(size 1.27 1.27)
+				)
+				(hide yes)
+			)
+		)
+		(property "Datasheet" "~"
+			(at 151.13 81.28 0)
+			(effects
+				(font
+					(size 1.27 1.27)
+				)
+				(hide yes)
+			)
+		)
+		(property "Description" "Resistor, small symbol"
+			(at 151.13 81.28 0)
+			(effects
+				(font
+					(size 1.27 1.27)
+				)
+				(hide yes)
+			)
+		)
+		(pin "1"
+		)
+		(pin "2"
+		)
+		(instances
+			(project "Mainboard"
+				(path "/351761a0-c9d1-4ae2-83c5-bde0949aa75f/00000000-0000-0000-0000-00005cec6281"
+					(reference "R1")
+					(unit 1)
+				)
+			)
+		)
+	)
+	(symbol
+		(lib_id "Device:R_Small")
 		(at 85.09 116.84 270)
 		(unit 1)
@@
 	)
 	(symbol
-		(lib_name "Mainboard:KMR231")
 		(lib_id "Mainboard:KMR231")
 		(at 40.64 78.74 0)
@@
 	)
 	(symbol
-		(lib_name "Mainboard:KMR231")
 		(lib_id "Mainboard:KMR231")
 		(at 40.64 60.96 0)
@@
 					(unit 1)
 				)
+			)
+		)
+	)
+	(symbol
+		(lib_id "Device:R_Small")
+		(at 151.13 83.82 270)
+		(unit 1)
+		(exclude_from_sim no)
+		(in_bom yes)
+		(on_board yes)
+		(dnp no)
+		(property "Reference" "R2"
+			(at 147.32 82.804 90)
+			(effects
+				(font
+					(size 1.27 1.27)
+				)
+			)
+		)
+		(property "Value" "0R"
+			(at 154.432 82.804 90)
+			(effects
+				(font
+					(size 1.27 1.27)
+				)
+			)
+		)
+		(property "Footprint" "Resistor_SMD:R_0603_1608Metric"
+			(at 151.13 83.82 0)
+			(effects
+				(font
+					(size 1.27 1.27)
+				)
+				(hide yes)
+			)
+		)
+		(property "Datasheet" "~"
+			(at 151.13 83.82 0)
+			(effects
+				(font
+					(size 1.27 1.27)
+				)
+				(hide yes)
+			)
+		)
+		(property "Description" "Resistor, small symbol"
+			(at 151.13 83.82 0)
+			(effects
+				(font
+					(size 1.27 1.27)
+				)
+				(hide yes)
+			)
+		)
+		(pin "1"
+		)
+		(pin "2"
+		)
+		(instances
+			(project "Mainboard"
+				(path "/351761a0-c9d1-4ae2-83c5-bde0949aa75f/00000000-0000-0000-0000-00005cec6281"
+					(reference "R2")
+					(unit 1)
+				)
